File: Compressor_Pedal.kicad_sch (KiCad schematic)
At the start: 20 parts, among them J1 InputJack, J2 OutputJack, J3 Sidechain, J4 Conn_01x03, U4 LM358, U5 LM358

Commit message: updates first build to add missing external mod switch - moving to v0.2
Parts:
- added JP3: Select, Connector_PinHeader_2.54mm:PinHeader_1x03_P2.54mm_Vertical, symbol Jumper:Jumper_3_Bridged12
- J1, J2, J3: footprint TestPoint:TestPoint_2Pads_Pitch5.08mm_Drill1.3mm -> Connector_PinHeader_2.54mm:PinHeader_1x02_P2.54mm_Vertical
- RV3: value A150k -> A200k; footprint Potentiometer_THT:Potentiometer_Alps_RK163_Single_Horizontal -> CustomLibrary:Potentiometer_Alps_RK163_Single_Horizontal_Pads_Only
- RV3: value A50k -> A20k; footprint Potentiometer_THT:Potentiometer_Alps_RK163_Single_Horizontal -> CustomLibrary:Potentiometer_Alps_RK163_Single_Horizontal_Pads_Only
Connections:
- net Volume Detector/signal_in: now also JP3.1 (A); no longer J3.2 (T), R19.2, U5.1
- new net: JP3.2 (C), R19.2, U5.1
- new net: J3.2 (T), JP3.3 (B)
Other:
- title: Compressor -> Compressor Pedal
- moved on the sheet: J3
Changed lines of the file:
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@@
   (paper "A4")
   (title_block
-    (title "Compressor")
-    (date "2023-05-27")
-    (rev "0.1")
+    (title "Compressor Pedal")
+    (date "2023-06-12")
+    (rev "0.2")
     (company "Jacob Miller")
     (comment 4 "All resistors are 1% unless noted")
+    (comment 9 "All resistors are 1% unless noted")
   )
   (junction (at 161.29 120.65) (diameter 0) (color 0 0 0 0)
@@
     (stroke (width 0) (type default))
   )
-  (wire (pts (xy 213.36 66.04) (xy 213.36 69.85))
+  (wire (pts (xy 227.33 66.04) (xy 227.33 69.85))
     (stroke (width 0) (type default))
   )
@@
     (stroke (width 0) (type default))
   )
-  (wire (pts (xy 207.01 77.47) (xy 207.01 63.5))
+  (wire (pts (xy 219.71 63.5) (xy 228.6 63.5))
     (stroke (width 0) (type default))
   )
@@
     (stroke (width 0) (type default))
   )
+  (wire (pts (xy 213.36 77.47) (xy 207.01 77.47))
+    (stroke (width 0) (type default))
+  )
   (wire (pts (xy 181.61 137.16) (xy 181.61 138.43))
     (stroke (width 0) (type default))
@@
     (stroke (width 0) (type default))
   )
+  (wire (pts (xy 213.36 67.31) (xy 213.36 77.47))
+    (stroke (width 0) (type default))
+  )
   (wire (pts (xy 153.67 90.17) (xy 161.29 90.17))
     (stroke (width 0) (type default))
@@
     (stroke (width 0) (type default))
   )
-  (wire (pts (xy 214.63 63.5) (xy 207.01 63.5))
-    (stroke (width 0) (type default))
-  )
   (wire (pts (xy 105.41 123.19) (xy 109.22 123.19))
     (stroke (width 0) (type default))
@@
     (stroke (width 0) (type default))
   )
-  (wire (pts (xy 214.63 66.04) (xy 213.36 66.04))
+  (wire (pts (xy 228.6 66.04) (xy 227.33 66.04))
     (stroke (width 0) (type default))
   )
@@
       (effects (font (size 1.27 1.27)) (justify right))
     )
-    (property "Value" "A150k" (at 184.15 128.27 90)
+    (property "Value" "A200k" (at 184.15 128.27 90)
       (effects (font (size 1.27 1.27)) (justify right))
     )
-    (property "Footprint" "Potentiometer_THT:Potentiometer_Alps_RK163_Single_Horizontal" (at 181.61 133.35 0)
+    (property "Footprint" "CustomLibrary:Potentiometer_Alps_RK163_Single_Horizontal_Pads_Only" (at 181.61 133.35 0)
       (effects (font (size 1.27 1.27)) hide)
     )
@@
       (effects (font (size 1.27 1.27)) (justify right))
     )
-    (property "Value" "A50k" (at 127 135.89 0)
+    (property "Value" "A20k" (at 127 135.89 0)
       (effects (font (size 1.27 1.27)) (justify right))
     )
-    (property "Footprint" "Potentiometer_THT:Potentiometer_Alps_RK163_Single_Horizontal" (at 125.73 134.62 0)
+    (property "Footprint" "CustomLibrary:Potentiometer_Alps_RK163_Single_Horizontal_Pads_Only" (at 125.73 134.62 0)
       (effects (font (size 1.27 1.27)) hide)
     )
@@
     )
   )
+  (symbol (lib_id "Jumper:Jumper_3_Bridged12") (at 213.36 63.5 0) (unit 1)
+    (in_bom yes) (on_board yes) (dnp no) (fields_autoplaced)
+    (property "Reference" "JP3" (at 213.36 59.6259 0)
+      (effects (font (size 1.27 1.27)))
+    )
+    (property "Value" "Select" (at 213.36 61.5469 0)
+      (effects (font (size 1.27 1.27)))
+    )
+    (property "Footprint" "Connector_PinHeader_2.54mm:PinHeader_1x03_P2.54mm_Vertical" (at 213.36 63.5 0)
+      (effects (font (size 1.27 1.27)) hide)
+    )
+    (property "Datasheet" "~" (at 213.36 63.5 0)
+      (effects (font (size 1.27 1.27)) hide)
+    )
+    (pin "1")
+    (pin "2")
+    (pin "3")
+    (instances
+      (project "Compressor_Pedal"
+        (path "/a4bfa001-f8c9-4599-807d-bef209d82349"
+          (reference "JP3") (unit 1)
+        )
+      )
+    )
+  )
   (symbol (lib_id "power:GNDA") (at 196.85 149.86 270) (unit 1)
     (in_bom yes) (on_board yes) (dnp no) (fields_autoplaced)
@@
       (effects (font (size 1.27 1.27)))
     )
-    (property "Footprint" "TestPoint:TestPoint_2Pads_Pitch5.08mm_Drill1.3mm" (at 208.28 123.19 0)
+    (property "Footprint" "Connector_PinHeader_2.54mm:PinHeader_1x02_P2.54mm_Vertical" (at 208.28 123.19 0)
       (effects (font (size 1.27 1.27)) hide)
     )
@@
     )
   )
-  (symbol (lib_id "power:GNDA") (at 213.36 69.85 0) (unit 1)
-    (in_bom yes) (on_board yes) (dnp no) (fields_autoplaced)
-    (property "Reference" "#PWR024" (at 213.36 76.2 0)
-      (effects (font (size 1.27 1.27)) hide)
-    )
-    (property "Value" "GNDA" (at 213.36 73.9855 0)
-      (effects (font (size 1.27 1.27)))
-    )
-    (property "Footprint" "" (at 213.36 69.85 0)
-      (effects (font (size 1.27 1.27)) hide)
-    )
-    (property "Datasheet" "" (at 213.36 69.85 0)
+  (symbol (lib_id "power:GNDA") (at 227.33 69.85 0) (unit 1)
+    (in_bom yes) (on_board yes) (dnp no) (fields_autoplaced)
+    (property "Reference" "#PWR024" (at 227.33 76.2 0)
+      (effects (font (size 1.27 1.27)) hide)
+    )
+    (property "Value" "GNDA" (at 227.33 73.9855 0)
+      (effects (font (size 1.27 1.27)))
+    )
+    (property "Footprint" "" (at 227.33 69.85 0)
+      (effects (font (size 1.27 1.27)) hide)
+    )
+    (property "Datasheet" "" (at 227.33 69.85 0)
       (effects (font (size 1.27 1.27)) hide)
     )
@@
       (effects (font (size 1.27 1.27)))
     )
-    (property "Footprint" "TestPoint:TestPoint_2Pads_Pitch5.08mm_Drill1.3mm" (at 100.33 123.19 0)
+    (property "Footprint" "Connector_PinHeader_2.54mm:PinHeader_1x02_P2.54mm_Vertical" (at 100.33 123.19 0)
       (effects (font (size 1.27 1.27)) hide)
     )
@@
     )
   )
-  (symbol (lib_name "AudioJack2_1") (lib_id "Connector_Audio:AudioJack2") (at 219.71 63.5 180) (unit 1)
+  (symbol (lib_name "AudioJack2_1") (lib_id "Connector_Audio:AudioJack2") (at 233.68 63.5 180) (unit 1)
     (in_bom yes) (on_board yes) (dnp no)
-    (property "Reference" "J3" (at 219.075 56.6801 0)
-      (effects (font (size 1.27 1.27)))
-    )
-    (property "Value" "Sidechain" (at 219.075 58.6011 0)
-      (effects (font (size 1.27 1.27)))
-    )
-    (property "Footprint" "TestPoint:TestPoint_2Pads_Pitch5.08mm_Drill1.3mm" (at 219.71 63.5 0)
-      (effects (font (size 1.27 1.27)) hide)
-    )
-    (property "Datasheet" "~" (at 219.71 63.5 0)
-      (effects (font (size 1.27 1.27)) hide)
-    )
+    (property "Reference" "J3" (at 233.045 56.6801 0)
+      (effects (font (size 1.27 1.27)))
+    )
+    (property "Value" "Sidechain" (at 233.045 58.6011 0)
+      (effects (font (size 1.27 1.27)))
+    )
+    (property "Footprint" "Connector_PinHeader_2.54mm:PinHeader_1x02_P2.54mm_Vertical" (at 233.68 63.5 0)
+      (effects (font (size 1.27 1.27)) hide)
+    )
+    (property "Datasheet" "~" (at 233.68 63.5 0)
+      (effects (font (size 1.27 1.27)) hide)
+    )
