File: volume_control.kicad_sch (KiCad schematic)
At the start: 25 parts, among them Q1 PN2222A, SW1 SW_DPDT_x2, U3 LM358

Commit message: sent for build
Parts:
- TP3: value cv_in -> CV1; footprint Connector_Pin:Pin_D1.3mm_L10.0mm_W3.5mm_Flat -> Connector_Pin:Pin_D0.9mm_L10.0mm_W2.4mm_FlatFork
- TP3: value cv_out -> CV2; footprint Connector_Pin:Pin_D1.3mm_L10.0mm_W3.5mm_Flat -> Connector_Pin:Pin_D0.9mm_L10.0mm_W2.4mm_FlatFork
Other:
- company: (none) -> Jacob Miller
- title: (none) -> Compressor
Changed lines of the file:
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@@
 (kicad_sch (version 20230121) (generator eeschema)
   (paper "A4")
+  (title_block
+    (title "Compressor")
+    (date "2023-05-27")
+    (rev "0.1")
+    (company "Jacob Miller")
+    (comment 1 "Volume Control Circuit")
+    (comment 4 "All resistors are 1% unless noted")
+    (comment 9 "All resistors are 1% unless noted")
+  )
   (junction (at 107.95 76.2) (diameter 0) (color 0 0 0 0)
   )
@@
       (effects (font (size 1.27 1.27)) (justify left))
     )
-    (property "Value" "cv_in" (at 109.347 66.5553 0)
+    (property "Value" "CV1" (at 109.347 66.5553 0)
       (effects (font (size 1.27 1.27)) (justify left))
     )
-    (property "Footprint" "Connector_Pin:Pin_D1.3mm_L10.0mm_W3.5mm_Flat" (at 113.03 68.58 0)
+    (property "Footprint" "Connector_Pin:Pin_D0.9mm_L10.0mm_W2.4mm_FlatFork" (at 113.03 68.58 0)
       (effects (font (size 1.27 1.27)) hide)
     )
@@
       (effects (font (size 1.27 1.27)) hide)
     )
-    (property "Description" "Threshold" (at 97.79 80.01 0)
+    (property "Description" "Ratio" (at 97.79 80.01 0)
       (effects (font (size 1.27 1.27)) (justify right))
     )
@@
       (effects (font (size 1.27 1.27)) (justify left))
     )
-    (property "Value" "cv_out" (at 161.417 72.9053 0)
+    (property "Value" "CV2" (at 161.417 72.9053 0)
       (effects (font (size 1.27 1.27)) (justify left))
     )
-    (property "Footprint" "Connector_Pin:Pin_D1.3mm_L10.0mm_W3.5mm_Flat" (at 165.1 74.93 0)
-      (effects (font (size 1.27 1.27)) hide)
-    )
+    (property "Footprint" "Connector_Pin:Pin_D0.9mm_L10.0mm_W2.4mm_FlatFork" (at 165.1 74.93 0)
+      (effects (font (size 1.27 1.27)) hide)
+    )

Commit message: updates first build to add missing external mod switch - moving to v0.2
Parts:
- R14: value 10k -> 1k
- RV3: footprint Potentiometer_THT:Potentiometer_Alps_RK163_Single_Horizontal -> CustomLibrary:Potentiometer_Alps_RK163_Single_Horizontal_Pads_Only
- SW1: footprint Button_Switch_THT:SW_NKK_GW12LJP -> CustomLibrary:SW_NKK_GW12LJP
Other:
- title: Compressor -> Compressor Pedal
Changed lines of the file:
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@@
   (paper "A4")
   (title_block
-    (title "Compressor")
-    (date "2023-05-27")
-    (rev "0.1")
+    (title "Compressor Pedal")
+    (date "2023-06-12")
+    (rev "0.2")
     (company "Jacob Miller")
     (comment 1 "Volume Control Circuit")
@@
       (effects (font (size 1.27 1.27)) (justify right))
     )
-    (property "Footprint" "Potentiometer_THT:Potentiometer_Alps_RK163_Single_Horizontal" (at 100.33 76.2 0)
+    (property "Footprint" "CustomLibrary:Potentiometer_Alps_RK163_Single_Horizontal_Pads_Only" (at 100.33 76.2 0)
       (effects (font (size 1.27 1.27)) hide)
     )
@@
       (effects (font (size 1.27 1.27)))
     )
-    (property "Footprint" "Button_Switch_THT:SW_NKK_GW12LJP" (at 195.58 78.74 0)
+    (property "Footprint" "CustomLibrary:SW_NKK_GW12LJP" (at 195.58 78.74 0)
       (effects (font (size 1.27 1.27)) hide)
     )
@@
       (effects (font (size 1.27 1.27)))
     )
-    (property "Footprint" "Button_Switch_THT:SW_NKK_GW12LJP" (at 195.58 113.03 0)
+    (property "Footprint" "CustomLibrary:SW_NKK_GW12LJP" (at 195.58 113.03 0)
       (effects (font (size 1.27 1.27)) hide)
     )
@@
       (effects (font (size 1.27 1.27)))
     )
-    (property "Value" "10k" (at 151.13 76.7621 90)
-      (effects (font (size 1.27 1.27)))
-    )
+    (property "Value" "1k" (at 151.13 76.7621 90)
+      (effects (font (size 1.27 1.27)))
+    )
