File: volume_detector.kicad_sch (KiCad schematic)
At the start: 23 parts, among them U1 LM358, U2 LM358

Commit message: schematic finished, begin layout
Parts:
- C1: footprint (none) -> Capacitor_THT:C_Radial_D5.0mm_H11.0mm_P2.00mm
- C2: footprint (none) -> Capacitor_THT:C_Disc_D5.0mm_W2.5mm_P2.50mm
- D1, D2, D3: footprint Diode_THT:D_DO-35_SOD27_P7.62mm_Horizontal -> Diode_THT:D_DO-35_SOD27_P2.54mm_Vertical_KathodeUp
- R1, R2, R3, R5, R6, R7, R8: footprint (none) -> Resistor_THT:R_Axial_DIN0207_L6.3mm_D2.5mm_P2.54mm_Vertical
- R4: value 100 -> 1k-4.7k; footprint (none) -> Resistor_THT:R_Axial_DIN0207_L6.3mm_D2.5mm_P2.54mm_Vertical
- R9: value 20k -> 33k; footprint (none) -> Resistor_THT:R_Axial_DIN0207_L6.3mm_D2.5mm_P2.54mm_Vertical
- RV1, RV2, RV3: footprint (none) -> Potentiometer_THT:Potentiometer_Alps_RK163_Single_Horizontal
- TP1: renamed from TP4; value ~ -> abs_s1; footprint (none) -> Connector_Pin:Pin_D1.3mm_L10.0mm_W3.5mm_Flat
- TP2: renamed from TP1; value Abs(Input) -> abs_out; footprint (none) -> Connector_Pin:Pin_D1.3mm_L10.0mm_W3.5mm_Flat
- TP3: renamed from TP2; footprint (none) -> Connector_Pin:Pin_D1.3mm_L10.0mm_W3.5mm_Flat
- TP4: renamed from TP3; footprint (none) -> Connector_Pin:Pin_D1.3mm_L10.0mm_W3.5mm_Flat
- U1, U2: footprint (none) -> Package_DIP:DIP-8_W7.62mm_Socket_LongPads
Connections:
- net at C1.1, R5.2, RV1.2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: now also RV1.3
- net at R4.2, RV2.2: now also RV2.3
- net Input renamed signal_in
- net Out renamed signal_out
- no-connect marks 2 -> 0
Other:
- note added: "Reference Voltage 9V * 33/(20+33) = 3.4V Assumes envelope voltage of less than 3.3V to allow turning off Or for 5V envelope 9V * 33/(20+47) = 5.3V"

Commit message: sent for build
Parts:
- TP1: value abs_s1 -> ABS1; footprint Connector_Pin:Pin_D1.3mm_L10.0mm_W3.5mm_Flat -> Connector_Pin:Pin_D0.9mm_L10.0mm_W2.4mm_FlatFork
- TP2: value abs_out -> ABS2; footprint Connector_Pin:Pin_D1.3mm_L10.0mm_W3.5mm_Flat -> Connector_Pin:Pin_D0.9mm_L10.0mm_W2.4mm_FlatFork
- TP3: value Envelope -> ENV; footprint Connector_Pin:Pin_D1.3mm_L10.0mm_W3.5mm_Flat -> Connector_Pin:Pin_D0.9mm_L10.0mm_W2.4mm_FlatFork
- TP4: value Threshold -> THR; footprint Connector_Pin:Pin_D1.3mm_L10.0mm_W3.5mm_Flat -> Connector_Pin:Pin_D0.9mm_L10.0mm_W2.4mm_FlatFork
Other:
- company: (none) -> Jacob Miller
- title: (none) -> Compressor
Changed lines of the file:
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@@
 (kicad_sch (version 20230121) (generator eeschema)
   (paper "A4")
+  (title_block
+    (title "Compressor")
+    (date "2023-05-27")
+    (rev "0.1")
+    (company "Jacob Miller")
+    (comment 1 "Volume Detection Circuit")
+    (comment 4 "All resistors are 1% unless noted")
+    (comment 9 "All resistors are 1% unless noted")
+  )
   (junction (at 97.79 106.68) (diameter 0) (color 0 0 0 0)
   )
@@
       (effects (font (size 1.27 1.27)) (justify left))
     )
-    (property "Value" "Envelope" (at 183.007 95.7653 0)
-      (effects (font (size 1.27 1.27)) (justify left))
-    )
-    (property "Footprint" "Connector_Pin:Pin_D1.3mm_L10.0mm_W3.5mm_Flat" (at 186.69 97.79 0)
+    (property "Value" "ENV" (at 183.007 95.7653 0)
+      (effects (font (size 1.27 1.27)) (justify left))
+    )
+    (property "Footprint" "Connector_Pin:Pin_D0.9mm_L10.0mm_W2.4mm_FlatFork" (at 186.69 97.79 0)
       (effects (font (size 1.27 1.27)) hide)
     )
@@
       (effects (font (size 1.27 1.27)) (justify left))
     )
-    (property "Value" "abs_out" (at 119.507 94.4953 0)
-      (effects (font (size 1.27 1.27)) (justify left))
-    )
-    (property "Footprint" "Connector_Pin:Pin_D1.3mm_L10.0mm_W3.5mm_Flat" (at 123.19 96.52 0)
+    (property "Value" "ABS2" (at 119.507 94.4953 0)
+      (effects (font (size 1.27 1.27)) (justify left))
+    )
+    (property "Footprint" "Connector_Pin:Pin_D0.9mm_L10.0mm_W2.4mm_FlatFork" (at 123.19 96.52 0)
       (effects (font (size 1.27 1.27)) hide)
     )
@@
       (effects (font (size 1.27 1.27)) (justify left))
     )
-    (property "Value" "Threshold" (at 218.567 79.2553 0)
-      (effects (font (size 1.27 1.27)) (justify left))
-    )
-    (property "Footprint" "Connector_Pin:Pin_D1.3mm_L10.0mm_W3.5mm_Flat" (at 222.25 81.28 0)
+    (property "Value" "THR" (at 218.567 79.2553 0)
+      (effects (font (size 1.27 1.27)) (justify left))
+    )
+    (property "Footprint" "Connector_Pin:Pin_D0.9mm_L10.0mm_W2.4mm_FlatFork" (at 222.25 81.28 0)
       (effects (font (size 1.27 1.27)) hide)
     )
@@
       (effects (font (size 1.27 1.27)) (justify left))
     )
-    (property "Value" "abs_s1" (at 80.137 94.4953 0)
-      (effects (font (size 1.27 1.27)) (justify left))
-    )
-    (property "Footprint" "Connector_Pin:Pin_D1.3mm_L10.0mm_W3.5mm_Flat" (at 83.82 96.52 0)
-      (effects (font (size 1.27 1.27)) hide)
-    )
+    (property "Value" "ABS1" (at 80.137 94.4953 0)
+      (effects (font (size 1.27 1.27)) (justify left))
+    )
+    (property "Footprint" "Connector_Pin:Pin_D0.9mm_L10.0mm_W2.4mm_FlatFork" (at 83.82 96.52 0)
+      (effects (font (size 1.27 1.27)) hide)
+    )

Commit message: updates first build to add missing external mod switch - moving to v0.2
Parts:
- R4: value 1k-4.7k -> 4.7k
- RV1, RV2, RV3: footprint Potentiometer_THT:Potentiometer_Alps_RK163_Single_Horizontal -> CustomLibrary:Potentiometer_Alps_RK163_Single_Horizontal_Pads_Only
Other:
- note added: "Reference Voltage 9V * 33/(20+33) = 3.4V Assumes envelope voltage of less than 3.3V to allow turning off Or for 5V envelope 9V * 15/(20+15) = 5.143V"
- note removed: "Reference Voltage 9V * 33/(20+33) = 3.4V Assumes envelope voltage of less than 3.3V to allow turning off Or for 5V envelope 9V * 33/(20+47) = 5.3V"
- title: Compressor -> Compressor Pedal
Changed lines of the file:
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@@
   (paper "A4")
   (title_block
-    (title "Compressor")
-    (date "2023-05-27")
-    (rev "0.1")
+    (title "Compressor Pedal")
+    (date "2023-06-12")
+    (rev "0.2")
     (company "Jacob Miller")
     (comment 1 "Volume Detection Circuit")
@@
     (effects (font (size 1.27 1.27)) (justify left top))
   )
+  (text_box "** Need to make Release last 10x longer"
+    (at 161.29 76.2 0) (size 27.94 8.89)
+    (stroke (width 0) (type default))
+    (fill (type none))
+    (effects (font (size 1.27 1.27)) (justify left top))
+  )
   (text_box "TI https://www.ti.com/lit/an/sboa068/sboa068.pdf Absolute Value Circui"
     (at 46.99 78.74 0) (size 78.74 67.31)
@@
     (effects (font (size 1.27 1.27)) (justify left top))
   )
-  (text "Reference Voltage\n9V * 33/(20+33) = 3.4V\nAssumes envelope voltage of less \nthan 3.3V to allow turning off\n\nOr for 5V envelope\n9V * 33/(20+47) = 5.3V"
+  (text "Reference Voltage\n9V * 33/(20+33) = 3.4V\nAssumes envelope voltage of less \nthan 3.3V to allow turning off\n\nOr for 5V envelope\n9V * 15/(20+15) = 5.143V"
     (at 218.44 73.66 0)
     (effects (font (size 1.27 1.27)) (justify left bottom))
@@
       (effects (font (size 1.27 1.27)) (justify right))
     )
-    (property "Footprint" "Potentiometer_THT:Potentiometer_Alps_RK163_Single_Horizontal" (at 195.58 106.68 0)
+    (property "Footprint" "CustomLibrary:Potentiometer_Alps_RK163_Single_Horizontal_Pads_Only" (at 195.58 106.68 0)
       (effects (font (size 1.27 1.27)) hide)
     )
@@
       (effects (font (size 1.27 1.27)))
     )
-    (property "Value" "1k-4.7k" (at 189.7921 118.11 90)
+    (property "Value" "4.7k" (at 189.7921 118.11 90)
       (effects (font (size 1.27 1.27)))
     )
@@
       (effects (font (size 1.27 1.27)))
     )
-    (property "Footprint" "Potentiometer_THT:Potentiometer_Alps_RK163_Single_Horizontal" (at 170.18 106.68 0)
+    (property "Footprint" "CustomLibrary:Potentiometer_Alps_RK163_Single_Horizontal_Pads_Only" (at 170.18 106.68 0)
       (effects (font (size 1.27 1.27)) hide)
     )
@@
       (effects (font (size 1.27 1.27)) (justify right))
     )
-    (property "Footprint" "Potentiometer_THT:Potentiometer_Alps_RK163_Single_Horizontal" (at 212.09 81.28 0)
-      (effects (font (size 1.27 1.27)) hide)
-    )
+    (property "Footprint" "CustomLibrary:Potentiometer_Alps_RK163_Single_Horizontal_Pads_Only" (at 212.09 81.28 0)
+      (effects (font (size 1.27 1.27)) hide)
+    )

Commit message: fix problem with external input
Parts:
- C1: value 1uF -> 22uF
- R4: value 4.7k -> 1.0k
Changed lines of the file:
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@@
       (effects (font (size 1.27 1.27)))
     )
-    (property "Value" "4.7k" (at 189.7921 118.11 90)
+    (property "Value" "1.0k" (at 189.7921 118.11 90)
       (effects (font (size 1.27 1.27)))
     )
@@
       (effects (font (size 1.27 1.27)) (justify left))
     )
-    (property "Value" "1uF" (at 183.769 107.4112 0)
+    (property "Value" "22uF" (at 183.769 107.4112 0)
       (effects (font (size 1.27 1.27)) (justify left))
     )
